File: roomba.sch (KiCad schematic (older format))
At the start: 10 parts, among them J1 Mini-DIN-7, J2 VIN, J3 VOUT, U1 LM317_3PinPackage, U2 NODEMCU_V2

Commit message: Updating circuit for Roomba PCB part placement complete
Adding ESP8266 part libraries
Parts:
- removed C1: 0.1µF, symbol Device:C
- removed C2: 47µF, symbol Device:CP
- removed J1: Mini-DIN-7, symbol Connector:Mini-DIN-7
- removed J2: VIN, symbol Connector:Conn_01x02_Female
- removed J3: VOUT, symbol Connector:Conn_01x02_Female
- removed JP1: (no value), symbol Device:Jumper_NC_Dual
- removed RV1: 10K, symbol Device:R_POT
- removed U1: LM317_3PinPackage, symbol Regulator_Linear:LM317_3PinPackage
- removed U2: NODEMCU_V2, Package_49x24.5x13mm, symbol nodemcu_v2:NODEMCU_V2
- added C1, C2, C3, C4: 10 uF, Capacitor_SMD:C_0805_2012Metric_Pad1.15x1.40mm_HandSolder, symbol Device:C_Small
- added J1: Conn_01x07_Male, Connector_PinHeader_2.54mm:PinHeader_1x07_P2.54mm_Vertical, symbol Connector:Conn_01x07_Male
- added J2: Conn_01x04_Female, Connector_PinSocket_2.54mm:PinSocket_1x04_P2.54mm_Vertical, symbol Connector:Conn_01x04_Female
- added R2, R3, R4, R5: 12K, Resistor_SMD:R_0805_2012Metric_Pad1.15x1.40mm_HandSolder, symbol Device:R_US
- added SW1: Reset, Button_Switch_SMD:SW_SPST_B3S-1000, symbol Switch:SW_Push
- added SW2: Flash, Button_Switch_SMD:SW_SPST_B3S-1000, symbol Switch:SW_Push
- added U1: TSR_1-2450, Converter_DCDC:Converter_DCDC_TRACO_TSR-1_THT, symbol Regulator_Switching:TSR_1-2450
- added U2: NCP1117-3.3_SOT223, Package_TO_SOT_SMD:SOT-223-3_TabPin2, symbol Regulator_Linear:NCP1117-3.3_SOT223
- added U3: TXB0104D, Package_SO:SOIC-14_3.9x8.7mm_P1.27mm, symbol Logic_LevelTranslator:TXB0104D
- added U4: ESP-12F, RF_Module:ESP-12E, symbol RF_Module:ESP-12F
- R1: value 200 -> 12K; footprint (none) -> Resistor_SMD:R_0805_2012Metric_Pad1.15x1.40mm_HandSolder
Connections:
- net labels added: +3.3V, GPIO0, GPIO2, LOCAL_BRC, LOCAL_RXD, LOCAL_TXD
- wire segments 68 -> 82
Other:
- note added: "+5V"
- note added: "--"
- note added: "2018/10/04"
- note added: "GND"
- note added: "Programming\nHeader"
- note added: "RXD"
- note added: "Roomba 560 ESP-Wifi"
- note added: "TXD"
- note removed: "1"
- note removed: "1-2: Normal boot\n2-3: Flash"
- note removed: "2018/08/29"
- note removed: "Buck Converter"
- note removed: "Note: Espressif CEO states I/O is 5V tolerant.\n Add level shifters for final design."
- note removed: "Roomba 560 ESP-Wifi Prototype"

Commit message: Routed PCB for Roomba
Parts:
- removed C4: 10 uF, Capacitor_SMD:C_0805_2012Metric_Pad1.15x1.40mm_HandSolder, symbol Device:C_Small
- removed J2: Conn_01x04_Female, Connector_PinSocket_2.54mm:PinSocket_1x04_P2.54mm_Vertical, symbol Connector:Conn_01x04_Female
- removed SW1: Reset, Button_Switch_SMD:SW_SPST_B3S-1000, symbol Switch:SW_Push
- removed SW2: Flash, Button_Switch_SMD:SW_SPST_B3S-1000, symbol Switch:SW_Push
Connections:
- wire segments 82 -> 67
Other:
- note removed: "+5V"
- note removed: "GND"
- note removed: "Programming\nHeader"
- note removed: "RXD"
- note removed: "TXD"
Changed lines of the file:
@@
 Wire Wire Line
 	7300 3550 7300 3850
-Wire Wire Line
-	6150 3850 7300 3850
 Connection ~ 7000 3650
 Text Label 7600 3650 0    50   ~ 0
 GPIO0
-Connection ~ 7300 3850
 Text Label 7600 3850 0    50   ~ 0
 GPIO2
@@
 	1850 4300 1850 4350
 Wire Wire Line
-	1850 4300 2650 4300
-Wire Wire Line
-	2650 4300 2650 4150
-Wire Wire Line
-	2650 3950 2650 3850
-Connection ~ 2650 3850
-Wire Wire Line
 	1200 5650 1200 5550
 Connection ~ 1200 5550
@@
 Wire Wire Line
 	2450 6000 1850 6000
-$Comp
-L Device:C_Small C4
-U 1 1 5BBA7B25
-P 2650 4050
-F 0 "C4" H 2742 4141 50  0000 L CNN
-F 1 "10 uF" H 2742 4050 50  0000 L CNN
-F 2 "Capacitor_SMD:C_0805_2012Metric_Pad1.15x1.40mm_HandSolder" H 2650 4050 50  0001 C CNN
-F 3 "~" H 2650 4050 50  0001 C CNN
-F 4 "25V" H 2742 3959 50  0000 L CNN "Voltage"
-	1    2650 4050
-	1    0    0    -1
-$EndComp
 $Comp
 L Device:C_Small C2
@@
 	1    0    0    -1
 $EndComp
-$Comp
-L Switch:SW_Push SW2
-U 1 1 5BBAE541
-P 8050 3650
-F 0 "SW2" H 7950 3750 50  0000 C CNN
-F 1 "Flash" H 8050 3550 50  0000 C CNN
-F 2 "Button_Switch_SMD:SW_SPST_B3S-1000" H 8050 3850 50  0001 C CNN
-F 3 "" H 8050 3850 50  0001 C CNN
-F 4 "B3S-1000" H 8050 3650 50  0001 C CNN "MFG_PN"
-	1    8050 3650
-	1    0    0    -1
-$EndComp
 Wire Wire Line
 	7000 3650 7850 3650
-Wire Wire Line
-	8250 3650 8350 3650
-Wire Wire Line
-	8350 3650 8350 3850
-Wire Wire Line
-	8350 3850 8350 4050
-$Comp
-L power:Earth #PWR020
-U 1 1 5BBB69AE
-P 8350 4050
-F 0 "#PWR020" H 8350 3800 50  0001 C CNN
-F 1 "Earth" H 8350 3900 50  0001 C CNN
-F 2 "" H 8350 4050 50  0001 C CNN
-F 3 "~" H 8350 4050 50  0001 C CNN
-	1    8350 4050
-	1    0    0    -1
-$EndComp
-$Comp
-L Switch:SW_Push SW1
-U 1 1 5BBB9752
-P 4450 4250
-F 0 "SW1" V 4600 4350 50  0000 C CNN
-F 1 "Reset" V 4400 4050 50  0000 C CNN
-F 2 "Button_Switch_SMD:SW_SPST_B3S-1000" H 4450 4450 50  0001 C CNN
-F 3 "" H 4450 4450 50  0001 C CNN
-F 4 "B3S-1000" V 4450 4250 50  0001 C CNN "MFG_PN"
-	1    4450 4250
-	0    -1   -1   0
-$EndComp
-Wire Wire Line
-	7300 3850 8350 3850
-Connection ~ 8350 3850
 Connection ~ 3800 3650
 Wire Wire Line
 	3800 3650 3800 3850
 Wire Wire Line
-	4300 3650 4450 3650
-Wire Wire Line
 	4300 3850 4950 3850
 Wire Wire Line
-	4450 4050 4450 3650
-Connection ~ 4450 3650
+	7300 3850 7850 3850
 Wire Wire Line
-	4450 3650 4950 3650
+	6150 3850 7300 3850
+Connection ~ 7300 3850
 Wire Wire Line
-	4450 4450 4450 4650
-$Comp
-L power:Earth #PWR012
-U 1 1 5BBCF3CA
-P 4450 4650
-F 0 "#PWR012" H 4450 4400 50  0001 C CNN
-F 1 "Earth" H 4450 4500 50  0001 C CNN
-F 2 "" H 4450 4650 50  0001 C CNN
-F 3 "~" H 4450 4650 50  0001 C CNN
-	1    4450 4650
-	1    0    0    -1
-$EndComp
-$Comp
-L Connector:Conn_01x04_Female J2
-U 1 1 5BBD583B
-P 2350 2800
-F 0 "J2" H 2244 2375 50  0000 C CNN
-F 1 "Conn_01x04_Female" H 2244 2466 50  0000 C CNN
-F 2 "Connector_PinSocket_2.54mm:PinSocket_1x04_P2.54mm_Vertical" H 2350 2800 50  0001 C CNN
-F 3 "~" H 2350 2800 50  0001 C CNN
-	1    2350 2800
-	-1   0    0    1
-$EndComp
-Wire Wire Line
-	2550 2600 2900 2600
-Wire Wire Line
-	2900 2600 2900 2500
-Wire Wire Line
-	2550 2700 2900 2700
-Wire Wire Line
-	2550 2800 2900 2800
-Wire Wire Line
-	2550 2900 2900 2900
-Wire Wire Line
-	2900 2900 2900 3000
-$Comp
-L power:Earth #PWR010
-U 1 1 5BBE496D
-P 2900 3000
-F 0 "#PWR010" H 2900 2750 50  0001 C CNN
-F 1 "Earth" H 2900 2850 50  0001 C CNN
-F 2 "" H 2900 3000 50  0001 C CNN
-F 3 "~" H 2900 3000 50  0001 C CNN
-	1    2900 3000
-	1    0    0    -1
-$EndComp
-$Comp
-L power:+5V #PWR09
-U 1 1 5BBE8442
-P 2900 2500
-F 0 "#PWR09" H 2900 2350 50  0001 C CNN
-F 1 "+5V" H 2915 2673 50  0000 C CNN
-F 2 "" H 2900 2500 50  0001 C CNN
-F 3 "" H 2900 2500 50  0001 C CNN
-	1    2900 2500
-	1    0    0    -1
-$EndComp
-Text Notes 1550 2850 0    50   Italic 0
-Programming\nHeader
-Text Label 2600 2700 0    50   Italic 0
-LOCAL_TXD
-Text Label 2600 2800 0    50   Italic 0
-LOCAL_RXD
-Text Notes 2150 2950 0    50   ~ 0
-GND
-Text Notes 2150 2850 0    50   ~ 0
-TXD
-Text Notes 2150 2750 0    50   ~ 0
-RXD
-Text Notes 2150 2650 0    50   ~ 0
-+5V
+	4300 3650 4950 3650
 $EndSCHEMATC

Commit message: Removed TXB0104, since it was garbling UART.  Instead added voltage divider on TXD from Roomba, and ran RXD and BRC to Roomba directly.
Parts:
- removed U3: TXB0104D, Package_SO:SOIC-14_3.9x8.7mm_P1.27mm, symbol Logic_LevelTranslator:TXB0104D
- added R6: 6.04K, Resistor_SMD:R_0805_2012Metric_Pad1.15x1.40mm_HandSolder, symbol Device:R_US
- added R7: 12K, Resistor_SMD:R_0805_2012Metric_Pad1.15x1.40mm_HandSolder, symbol Device:R_US
Connections:
- wire segments 67 -> 64
Changed lines of the file:
@@
 	1850 4150 1850 4300
-$Comp
-L Logic_LevelTranslator:TXB0104D U3
-U 1 1 5BB7A4D3
-P 5450 1750
-F 0 "U3" H 5200 2450 50  0000 C CNN
-F 1 "TXB0104D" H 5700 1100 50  0000 C CNN
-F 2 "Package_SO:SOIC-14_3.9x8.7mm_P1.27mm" H 5450 1000 50  0001 C CNN
-F 3 "http://www.ti.com/lit/ds/symlink/txb0104.pdf" H 5560 1845 50  0001 C CNN
-	1    5450 1750
-	1    0    0    -1
-$EndComp
-$Comp
-L power:+5V #PWR017
-U 1 1 5BB7A5AB
-P 5600 850
-F 0 "#PWR017" H 5600 700 50  0001 C CNN
-F 1 "+5V" H 5615 1023 50  0000 C CNN
-F 2 "" H 5600 850 50  0001 C CNN
-F 3 "" H 5600 850 50  0001 C CNN
-	1    5600 850
-	1    0    0    -1
-$EndComp
 $Comp
 L power:+3.3V #PWR015
@@
 Wire Wire Line
 	5550 3450 5550 3250
-$Comp
-L power:+3.3V #PWR013
-U 1 1 5BB7DFB5
-P 5350 850
-F 0 "#PWR013" H 5350 700 50  0001 C CNN
-F 1 "+3.3V" H 5365 1023 50  0000 C CNN
-F 2 "" H 5350 850 50  0001 C CNN
-F 3 "" H 5350 850 50  0001 C CNN
-	1    5350 850
-	1    0    0    -1
-$EndComp
-Wire Wire Line
-	5350 1050 5350 850
-Wire Wire Line
-	5550 1050 5550 950
-Wire Wire Line
-	5550 950  5600 950
-Wire Wire Line
-	5600 950  5600 850
-Wire Wire Line
-	5850 1650 6400 1650
-Text Label 5950 1650 0    50   Italic 0
+Text Label 5950 2200 0    50   Italic 0
 ROOMBA_RXD
-Wire Wire Line
-	5850 1450 6400 1450
-Text Label 5950 1450 0    50   Italic 0
+Text Label 5950 1000 0    50   Italic 0
 ROOMBA_TXD
-Wire Wire Line
-	5850 1850 6400 1850
-Text Label 5950 1850 0    50   Italic 0
+Text Label 5950 2400 0    50   Italic 0
 ROOMBA_BRC
-Wire Wire Line
-	4250 1650 5050 1650
-Text Label 4300 1650 0    50   ~ 0
+Text Label 4300 2200 0    50   ~ 0
 LOCAL_TXD
-Wire Wire Line
-	4250 1450 5050 1450
 Text Label 4300 1450 0    50   ~ 0
 LOCAL_RXD
-Wire Wire Line
-	4250 1850 5050 1850
-Text Label 4300 1850 0    50   ~ 0
+Text Label 4300 2400 0    50   ~ 0
 LOCAL_BRC
-$Comp
-L power:Earth #PWR014
-U 1 1 5BB8B769
-P 5450 2700
-F 0 "#PWR014" H 5450 2450 50  0001 C CNN
-F 1 "Earth" H 5450 2550 50  0001 C CNN
-F 2 "" H 5450 2700 50  0001 C CNN
-F 3 "~" H 5450 2700 50  0001 C CNN
-	1    5450 2700
-	1    0    0    -1
-$EndComp
-Wire Wire Line
-	5450 2450 5450 2700
 $Comp
 L Connector:Conn_01x07_Male J1
@@
 Wire Wire Line
 	4300 3650 4950 3650
+Wire Wire Line
+	4250 2200 6400 2200
+Wire Wire Line
+	4250 2400 6400 2400
+$Comp
+L Device:R_US R7
+U 1 1 5BCD7E32
+P 5450 1650
+F 0 "R7" H 5550 1550 50  0000 C CNN
+F 1 "12K" H 5550 1800 50  0000 C CNN
+F 2 "Resistor_SMD:R_0805_2012Metric_Pad1.15x1.40mm_HandSolder" V 5490 1640 50  0001 C CNN
+F 3 "~" H 5450 1650 50  0001 C CNN
+	1    5450 1650
+	-1   0    0    1
+$EndComp
+$Comp
+L power:Earth #PWR0101
+U 1 1 5BCDCD68
+P 5450 1900
+F 0 "#PWR0101" H 5450 1650 50  0001 C CNN
+F 1 "Earth" H 5450 1750 50  0001 C CNN
+F 2 "" H 5450 1900 50  0001 C CNN
+F 3 "~" H 5450 1900 50  0001 C CNN
+	1    5450 1900
+	1    0    0    -1
+$EndComp
+Wire Wire Line
+	5450 1800 5450 1900
+$Comp
+L Device:R_US R6
+U 1 1 5BCDDD61
+P 5450 1250
+F 0 "R6" H 5550 1150 50  0000 C CNN
+F 1 "6.04K" H 5550 1400 50  0000 C CNN
+F 2 "Resistor_SMD:R_0805_2012Metric_Pad1.15x1.40mm_HandSolder" V 5490 1240 50  0001 C CNN
+F 3 "~" H 5450 1250 50  0001 C CNN
+	1    5450 1250
+	-1   0    0    1
+$EndComp
+Wire Wire Line
+	5450 1400 5450 1450
+Wire Wire Line
+	5450 1000 5450 1100
+Wire Wire Line
+	5450 1000 6400 1000
+Wire Wire Line
+	4250 1450 5450 1450
+Connection ~ 5450 1450
+Wire Wire Line
+	5450 1450 5450 1500
 $EndSCHEMATC

Commit message: Updating Roomba project to use buttons for reset/programming. Removing 5V to 3.3V translator in favor of voltage divider. Removing 5V to 3.3V regulator and going directly from BATT to 3.3V.
Parts:
- removed C2: 10 uF, Capacitor_SMD:C_0805_2012Metric_Pad1.15x1.40mm_HandSolder, symbol Device:C_Small
- removed U1: TSR_1-2450, Converter_DCDC:Converter_DCDC_TRACO_TSR-1_THT, symbol Regulator_Switching:TSR_1-2450
- removed U2: NCP1117-3.3_SOT223, Package_TO_SOT_SMD:SOT-223-3_TabPin2, symbol Regulator_Linear:NCP1117-3.3_SOT223
- added R8, R9: 470, Resistor_SMD:R_0805_2012Metric_Pad1.15x1.40mm_HandSolder, symbol Device:R_US
- added SW1, SW2: SW_Push, pts820:PTS820, symbol Switch:SW_Push
- added U1: TSR_1-2433, Converter_DCDC:Converter_DCDC_TRACO_TSR-1_THT, symbol Regulator_Switching:TSR_1-2433
Connections:
- net labels removed: +5V
- no-connect marks 0 -> 12
Other:
- note added: "A"
- note removed: "--"
Changed lines of the file:
@@
-	1    0    0    -1
-$EndComp
-$Comp
-L power:+5V #PWR08
-U 1 1 5B887698
-P 2650 3650
-F 0 "#PWR08" H 2650 3500 50  0001 C CNN
-F 1 "+5V" H 2665 3823 50  0000 C CNN
-F 2 "" H 2650 3650 50  0001 C CNN
-F 3 "" H 2650 3650 50  0001 C CNN
-	1    2650 3650
 	1    0    0    -1
 $EndComp
@@
 Roomba 560 ESP-Wifi
 Text Notes 10600 7650 0    50   ~ 0
---
+A
 Text Notes 7000 7100 0    50   ~ 0
 Drawn by: Matthew A Sparks
@@
 	1200 1400 1500 1400
 Wire Wire Line
-	1200 1500 1500 1500
-Wire Wire Line
-	1500 1500 1500 1400
-Connection ~ 1500 1400
-Wire Wire Line
 	1500 1900 1500 2000
 Wire Wire Line
@@
 Text Label 1750 1700 0    50   ~ 0
 ROOMBA_TXD
-$Comp
-L Regulator_Switching:TSR_1-2450 U1
-U 1 1 5BB72BEF
-P 1850 3950
-F 0 "U1" H 1600 4300 50  0000 C CNN
-F 1 "TSR_1-2450" H 1850 4226 50  0000 C CNN
-F 2 "Converter_DCDC:Converter_DCDC_TRACO_TSR-1_THT" H 1850 3800 50  0001 L CIN
-F 3 "http://www.tracopower.com/products/tsr1.pdf" H 1850 3950 50  0001 C CNN
-	1    1850 3950
-	1    0    0    -1
-$EndComp
 Wire Wire Line
 	1050 3850 1450 3850
@@
 	7000 3000 7000 3250
 $Comp
-L Regulator_Linear:NCP1117-3.3_SOT223 U2
-U 1 1 5BB8FA5F
-P 1850 5550
-F 0 "U2" H 1500 5800 50  0000 C CNN
-F 1 "NCP1117-3.3_SOT223" H 1850 5701 50  0000 C CNN
-F 2 "Package_TO_SOT_SMD:SOT-223-3_TabPin2" H 1850 5750 50  0001 C CNN
-F 3 "http://www.onsemi.com/pub_link/Collateral/NCP1117-D.PDF" H 1950 5300 50  0001 C CNN
-	1    1850 5550
-	1    0    0    -1
-$EndComp
-$Comp
-L power:Earth #PWR06
-U 1 1 5BB91071
-P 1850 6050
-F 0 "#PWR06" H 1850 5800 50  0001 C CNN
-F 1 "Earth" H 1850 5900 50  0001 C CNN
-F 2 "" H 1850 6050 50  0001 C CNN
-F 3 "~" H 1850 6050 50  0001 C CNN
-	1    1850 6050
-	1    0    0    -1
-$EndComp
-Wire Wire Line
-	1850 5850 1850 6000
-$Comp
-L power:+5V #PWR02
-U 1 1 5BB925AF
-P 1200 5350
-F 0 "#PWR02" H 1200 5200 50  0001 C CNN
-F 1 "+5V" H 1215 5523 50  0000 C CNN
-F 2 "" H 1200 5350 50  0001 C CNN
-F 3 "" H 1200 5350 50  0001 C CNN
-	1    1200 5350
-	1    0    0    -1
-$EndComp
-Wire Wire Line
-	1200 5550 1200 5350
-$Comp
-L power:+3.3V #PWR07
-U 1 1 5BB930C9
-P 2450 5350
-F 0 "#PWR07" H 2450 5200 50  0001 C CNN
-F 1 "+3.3V" H 2465 5523 50  0000 C CNN
-F 2 "" H 2450 5350 50  0001 C CNN
-F 3 "" H 2450 5350 50  0001 C CNN
-	1    2450 5350
-	1    0    0    -1
-$EndComp
-Wire Wire Line
-	1200 5550 1550 5550
-Wire Wire Line
-	2150 5550 2450 5550
-Wire Wire Line
-	2450 5350 2450 5550
-$Comp
 L Device:C_Small C1
 U 1 1 5BB9991F
@@
 	1850 4300 1850 4350
 Wire Wire Line
-	1200 5650 1200 5550
-Connection ~ 1200 5550
-Wire Wire Line
-	1200 5850 1200 6000
-Wire Wire Line
-	1200 6000 1850 6000
-Connection ~ 1850 6000
-Wire Wire Line
-	1850 6000 1850 6050
-Wire Wire Line
-	2450 5650 2450 5550
-Connection ~ 2450 5550
-Wire Wire Line
-	2450 5850 2450 6000
-Wire Wire Line
-	2450 6000 1850 6000
-$Comp
-L Device:C_Small C2
-U 1 1 5BBABA07
-P 1200 5750
-F 0 "C2" H 1292 5841 50  0000 L CNN
-F 1 "10 uF" H 1292 5750 50  0000 L CNN
-F 2 "Capacitor_SMD:C_0805_2012Metric_Pad1.15x1.40mm_HandSolder" H 1200 5750 50  0001 C CNN
-F 3 "~" H 1200 5750 50  0001 C CNN
-F 4 "25V" H 1292 5659 50  0000 L CNN "Voltage"
-	1    1200 5750
-	1    0    0    -1
-$EndComp
+	2650 3950 2650 3850
+Wire Wire Line
+	2650 4150 2650 4300
 $Comp
 L Device:C_Small C3
 U 1 1 5BBACEE9
-P 2450 5750
-F 0 "C3" H 2542 5841 50  0000 L CNN
-F 1 "10 uF" H 2542 5750 50  0000 L CNN
-F 2 "Capacitor_SMD:C_0805_2012Metric_Pad1.15x1.40mm_HandSolder" H 2450 5750 50  0001 C CNN
-F 3 "~" H 2450 5750 50  0001 C CNN
-F 4 "25V" H 2542 5659 50  0000 L CNN "Voltage"
-	1    2450 5750
-	1    0    0    -1
-$EndComp
-Wire Wire Line
-	7000 3650 7850 3650
+P 2650 4050
+F 0 "C3" H 2742 4141 50  0000 L CNN
+F 1 "10 uF" H 2742 4050 50  0000 L CNN
+F 2 "Capacitor_SMD:C_0805_2012Metric_Pad1.15x1.40mm_HandSolder" H 2650 4050 50  0001 C CNN
+F 3 "~" H 2650 4050 50  0001 C CNN
+F 4 "25V" H 2742 3959 50  0000 L CNN "Voltage"
+	1    2650 4050
+	1    0    0    -1
+$EndComp
 Connection ~ 3800 3650
 Wire Wire Line
 	3800 3650 3800 3850
-Wire Wire Line
-	4300 3850 4950 3850
 Wire Wire Line
 	7300 3850 7850 3850
@@
 	6150 3850 7300 3850
 Connection ~ 7300 3850
-Wire Wire Line
-	4300 3650 4950 3650
 Wire Wire Line
 	4250 2200 6400 2200
@@
 $EndComp
 $Comp
+L Device:R_US R6
+U 1 1 5BCDDD61
+P 5450 1250
+F 0 "R6" H 5550 1150 50  0000 C CNN
+F 1 "6.04K" H 5550 1400 50  0000 C CNN
+F 2 "Resistor_SMD:R_0805_2012Metric_Pad1.15x1.40mm_HandSolder" V 5490 1240 50  0001 C CNN
+F 3 "~" H 5450 1250 50  0001 C CNN
+	1    5450 1250
+	-1   0    0    1
+$EndComp
+Wire Wire Line
+	5450 1400 5450 1450
+Wire Wire Line
+	5450 1000 5450 1100
+Wire Wire Line
+	5450 1000 6400 1000
+Wire Wire Line
+	4250 1450 5450 1450
+Connection ~ 5450 1450
+Wire Wire Line
+	5450 1450 5450 1500
+Wire Wire Line
+	1200 1500 1800 1500
+$Comp
+L Switch:SW_Push SW1
+U 1 1 5BDA94D1
+P 4350 4250
+F 0 "SW1" V 4304 4398 50  0000 L CNN
+F 1 "SW_Push" V 4395 4398 50  0000 L CNN
+F 2 "pts820:PTS820" H 4350 4450 50  0001 C CNN
+F 3 "" H 4350 4450 50  0001 C CNN
+	1    4350 4250
+	0    1    1    0
+$EndComp
+$Comp
+L Switch:SW_Push SW2
+U 1 1 5BDA95B5
+P 8050 3950
+F 0 "SW2" V 8004 4098 50  0000 L CNN
+F 1 "SW_Push" V 8095 4098 50  0000 L CNN
+F 2 "pts820:PTS820" H 8050 4150 50  0001 C CNN
+F 3 "" H 8050 4150 50  0001 C CNN
+	1    8050 3950
+	0    1    1    0
+$EndComp
+$Comp
+L Device:R_US R8
+U 1 1 5BDAA6FA
+P 4350 4700
+F 0 "R8" H 4450 4600 50  0000 C CNN
+F 1 "470" H 4450 4850 50  0000 C CNN
+F 2 "Resistor_SMD:R_0805_2012Metric_Pad1.15x1.40mm_HandSolder" V 4390 4690 50  0001 C CNN
+F 3 "~" H 4350 4700 50  0001 C CNN
+	1    4350 4700
+	-1   0    0    1
+$EndComp
+$Comp
+L Device:R_US R9
+U 1 1 5BDAB8A8
+P 8050 4400
+F 0 "R9" H 8150 4300 50  0000 C CNN
+F 1 "470" H 8150 4550 50  0000 C CNN
+F 2 "Resistor_SMD:R_0805_2012Metric_Pad1.15x1.40mm_HandSolder" V 8090 4390 50  0001 C CNN
+F 3 "~" H 8050 4400 50  0001 C CNN
+	1    8050 4400
+	-1   0    0    1
+$EndComp
+$Comp
+L power:Earth #PWR0103
+U 1 1 5BDADB60
+P 4350 5100
+F 0 "#PWR0103" H 4350 4850 50  0001 C CNN
+F 1 "Earth" H 4350 4950 50  0001 C CNN
+F 2 "" H 4350 5100 50  0001 C CNN
+F 3 "~" H 4350 5100 50  0001 C CNN
+	1    4350 5100
+	1    0    0    -1
+$EndComp
+Wire Wire Line
+	4350 4850 4350 5100
+$Comp
+L power:Earth #PWR0104
+U 1 1 5BDAECE0
+P 8050 4800
+F 0 "#PWR0104" H 8050 4550 50  0001 C CNN
+F 1 "Earth" H 8050 4650 50  0001 C CNN
+F 2 "" H 8050 4800 50  0001 C CNN
+F 3 "~" H 8050 4800 50  0001 C CNN
+	1    8050 4800
+	1    0    0    -1
+$EndComp
+Wire Wire Line
+	8050 4550 8050 4800
+Wire Wire Line
+	8050 4250 8050 4150
+Wire Wire Line
+	8050 3750 8050 3650
+Wire Wire Line
+	7000 3650 8050 3650
+Wire Wire Line
+	4350 4450 4350 4550
+NoConn ~ 4950 4050
+NoConn ~ 4950 4250
+NoConn ~ 4950 4350
+NoConn ~ 4950 4450
+NoConn ~ 4950 4550
+NoConn ~ 4950 4650
+NoConn ~ 4950 4750
+NoConn ~ 6150 4450
+NoConn ~ 6150 4350
+NoConn ~ 6150 4250
+NoConn ~ 6150 4150
+NoConn ~ 6150 4050
+$Comp
 L power:Earth #PWR0101
 U 1 1 5BCDCD68
@@
 	5450 1800 5450 1900
 $Comp
-L Device:R_US R6
-U 1 1 5BCDDD61
-P 5450 1250
-F 0 "R6" H 5550 1150 50  0000 C CNN
-F 1 "6.04K" H 5550 1400 50  0000 C CNN
-F 2 "Resistor_SMD:R_0805_2012Metric_Pad1.15x1.40mm_HandSolder" V 5490 1240 50  0001 C CNN
-F 3 "~" H 5450 1250 50  0001 C CNN
-	1    5450 1250
-	-1   0    0    1
-$EndComp
-Wire Wire Line
-	5450 1400 5450 1450
-Wire Wire Line
-	5450 1000 5450 1100
-Wire Wire Line
-	5450 1000 6400 1000
-Wire Wire Line
-	4250 1450 5450 1450
-Connection ~ 5450 1450
-Wire Wire Line
-	5450 1450 5450 1500
+L Regulator_Switching:TSR_1-2433 U1
+U 1 1 5BDCB2FC
+P 1850 3950
+F 0 "U1" H 1850 4317 50  0000 C CNN
+F 1 "TSR_1-2433" H 1850 4226 50  0000 C CNN
+F 2 "Converter_DCDC:Converter_DCDC_TRACO_TSR-1_THT" H 1850 3800 50  0001 L CIN
+F 3 "http://www.tracopower.com/products/tsr1.pdf" H 1850 3950 50  0001 C CNN
+	1    1850 3950
+	1    0    0    -1
+$EndComp
+$Comp
+L power:+3.3V #PWR0102
+U 1 1 5BDD02DB
+P 2650 3650
+F 0 "#PWR0102" H 2650 3500 50  0001 C CNN
+F 1 "+3.3V" H 2665 3823 50  0000 C CNN
+F 2 "" H 2650 3650 50  0001 C CNN
+F 3 "" H 2650 3650 50  0001 C CNN
+	1    2650 3650
+	1    0    0    -1
+$EndComp
+Connection ~ 2650 3850
+Wire Wire Line
+	1850 4300 2650 4300
+Wire Wire Line
+	1800 1500 1800 1300
+$Comp
+L power:+3.3V #PWR0105
+U 1 1 5BDD6910
+P 1800 1300
+F 0 "#PWR0105" H 1800 1150 50  0001 C CNN
+F 1 "+3.3V" H 1815 1473 50  0000 C CNN
+F 2 "" H 1800 1300 50  0001 C CNN
+F 3 "" H 1800 1300 50  0001 C CNN
+	1    1800 1300
+	1    0    0    -1
+$EndComp
+Wire Wire Line
+	4300 3850 4950 3850
+Wire Wire Line
+	4300 3650 4500 3650
+Wire Wire Line
+	4350 4050 4350 3950
+Wire Wire Line
+	4350 3950 4500 3950
+Wire Wire Line
+	4500 3950 4500 3650
+Connection ~ 4500 3650
+Wire Wire Line
+	4500 3650 4950 3650
 $EndSCHEMATC
